Commit message: DDD

File: src/delivery_description/urdf/wheels.xacro (robot description, xacro)
@@ -4,5 +4,5 @@
     <link name="left_wheel_link"/>
     <link name="right_wheel_link"/>
-    <joint name="left_wheel_joint" type="continuous">
+    <joint name="left_wheel_joint" type="fixed">
       <parent link="base_link"/>
       <child link="left_wheel_link"/>
@@ -10,5 +10,5 @@
       <axis xyz="0 1 0"/>
     </joint>
-    <joint name="right_wheel_joint" type="continuous">
+    <joint name="right_wheel_joint" type="fixed">
       <parent link="base_link"/>
       <child link="right_wheel_link"/>
