Commit message: tune nav2 params

File: src/delivery_description/urdf/delivery.urdf.xacro (robot description, xacro)
@@ -3,12 +3,17 @@
   <!-- include utils FIRST -->
   <xacro:include filename="$(find delivery_description)/urdf/utils.xacro"/>
-  <!-- params (meters) -->
+  <!-- robot size -->
+  <xacro:property name="robot_length" value="0.40"/>
+  <xacro:property name="robot_width"  value="0.30"/>
+  <!-- wheel params -->
   <xacro:property name="wheel_radius" value="0.033"/>
-  <xacro:property name="wheel_separation" value="0.36"/>
+  <xacro:property name="wheel_separation" value="0.355"/>
   <xacro:property name="wheel_y" value="${wheel_separation/2.0}"/>
-  <!-- LiDAR pose (meters + degrees) -->
-  <xacro:property name="lidar_x" value="0.15"/>
+  <xacro:property name="wheel_x" value="0.0"/>
+  <xacro:property name="wheel_axis_z" value="-0.017"/>
+  <!-- LiDAR pose -->
+  <xacro:property name="lidar_x" value="0.1125"/>
   <xacro:property name="lidar_y" value="0.0"/>
-  <xacro:property name="lidar_z" value="0.20"/>
+  <xacro:property name="lidar_z" value="0.245"/>
   <!-- degrees only -->
   <xacro:property name="lidar_roll_deg"  value="0"/>
@@ -22,11 +27,16 @@
   <!-- call macros -->
   <xacro:base/>
-    <!-- ✅ IMU TF: เรียกหลัง base_link ถูกสร้างแล้ว -->
+  <!-- IMU -->
   <xacro:add_imu
     parent="base_link"
     imu_name="bno055"
-    xyz="0.10 0.00 0.08"
+    xyz="-0.05 0.0 0.02"
     rpy="0 0 0"/>
-  <xacro:wheels wheel_y="${wheel_y}" wheel_radius="${wheel_radius}"/>
+  <!-- wheels -->
+  <xacro:wheels
+    wheel_x="${wheel_x}"
+    wheel_y="${wheel_y}"
+    wheel_axis_z="${wheel_axis_z}"/>
+  <!-- lidar -->
   <xacro:lidar
     lidar_x="${lidar_x}" lidar_y="${lidar_y}" lidar_z="${lidar_z}"

File: src/delivery_description/urdf/lidar.xacro (robot description, xacro)
@@ -1,5 +1,4 @@
 <?xml version="1.0"?>
 <robot xmlns:xacro="http://www.ros.org/wiki/xacro">
-  <!-- uses D2R from utils.xacro -->
   <xacro:macro name="lidar" params="lidar_x lidar_y lidar_z lidar_roll_deg lidar_pitch_deg lidar_yaw_deg">
     <link name="lidar_link"/>

File: src/delivery_description/urdf/wheels.xacro (robot description, xacro)
@@ -1,5 +1,5 @@
 <?xml version="1.0"?>
 <robot xmlns:xacro="http://www.ros.org/wiki/xacro">
-  <xacro:macro name="wheels" params="wheel_y wheel_radius">
+  <xacro:macro name="wheels" params="wheel_x wheel_y wheel_axis_z">
     <link name="left_wheel_link"/>
     <link name="right_wheel_link"/>
@@ -7,5 +7,5 @@
       <parent link="base_link"/>
       <child link="left_wheel_link"/>
-      <origin xyz="0 ${wheel_y} ${wheel_radius}" rpy="0 0 0"/>
+      <origin xyz="${wheel_x} ${wheel_y} ${wheel_axis_z}" rpy="0 0 0"/>
       <axis xyz="0 1 0"/>
     </joint>
@@ -13,5 +13,5 @@
       <parent link="base_link"/>
       <child link="right_wheel_link"/>
-      <origin xyz="0 -${wheel_y} ${wheel_radius}" rpy="0 0 0"/>
+      <origin xyz="${wheel_x} -${wheel_y} ${wheel_axis_z}" rpy="0 0 0"/>
       <axis xyz="0 1 0"/>
     </joint>
